File: KiCad/KiCad.kicad_sch (KiCad schematic)
At the start: 4 parts, among them SW1 SW_Push, SW2 SW_Push, SW3 SW_Push, U1 MOUDLE-SEEEDUINO-XIAO

Commit message: Add rotary encoder and redesigned the case.
Parts:
- added SW6: RotaryEncoder_Switch, Rotary_Encoder:RotaryEncoder_Alps_EC11E-Switch_Vertical_H20mm_MountingHoles, symbol Device:RotaryEncoder_Switch
Connections:
- net GND: now also SW6.C, SW6.S1
- net at U1.10 (PA5_A9_D9_MISO): no longer SW2.1
- net at U1.11 (PA6_A10_D10_MOSI): no longer SW1.1
- net at U1.2 (PA4_A1_D1): now also SW6.A
- net at U1.3 (PA10_A2_D2): now also SW6.B
- net at U1.4 (PA11_A3_D3): now also SW6.S2
- net at U1.5 (PA8_A4_D4_SDA): now also SW1.1
- net at U1.6 (PA9_A5_D5_SCL): now also SW2.1
- net at U1.7 (PB08_A6_D6_TX): now also SW3.1
- net at U1.9 (PA7_A8_D8_SCK): no longer SW3.1
